File: electrical_cable_distributor/ecd.brd (EAGLE design)
At the start: 4 parts

Commit message: added missing dimentions drawing
Parts:
- moved X1 32.7 mm to (6.39, 19.4)
- moved X2 32.7 mm to (19.4, 32.4)
- moved X3 32.7 mm to (32.4, 19.4)
- moved X4 32.7 mm to (19.4, 6.41)
Other:
- board outline added: 38.8 x 38.9 mm
