File: led_power_decoupling/led_power_decoupling.sch (EAGLE design)
At the start: 0 parts

Commit message: LED power decoupling board
Parts:
- added C1, C4: 10mF, rcl:CPOL-EUE7.5-16
- added C2, C5: 10mF (low. imp.), rcl:CPOL-EUE7.5-18
- added C3, C6: 22mF, rcl:CPOL-EUE10-25
- added X1: out 1, con-ptr500:AK500/2
- added X2: out 2, con-ptr500:AK500/2
- added X3: input, con-ptr500:AK500/2
Connections:
- new net +12V: C1.+, C2.+, C3.+, C4.+, C5.+, C6.+, X1-1.KL, X2-2.KL, X3-1.KL
- new net 0V: C1.-, C2.-, C3.-, C4.-, C5.-, C6.-, X1-2.KL, X2-1.KL, X3-2.KL
