File: koala_buzzer/hw/satellite_hw.kicad_pcb (KiCad board)
At the start: 2 copper layers, 43.7 x 21.1 mm, 21 parts, among them J1 solar 1, J2 solar 2, J3 solar 3, J4 solar 4, Q1 2N7002, U1 AP3015, U2 ATtiny13-20SU

Commit message: updated values for capacitors for DC/DC
Parts:
- C1: value 4.7µF -> 10µF
- C2: value 20µF -> 1µF
