File: pwm_light_ctrl/hw/board/board.kicad_sch (KiCad schematic)
At the start: 7 parts, among them J1 input, J2 output LED, Q1 IRF530, U1 L78L05_TO92

Commit message: * IRF530 -> IRFZ44N (for higher currents with less losses) * fixed resistors labeling * added PNP to driver MOSFET
Parts:
- added Q2: PN2222A, Package_TO_SOT_THT:TO-92_Inline, symbol Transistor_BJT:PN2222A
- added R2, R3: 1k, symbol Device:R
- PR1: renamed from 100k2; value R_Potentiometer -> 100k
- Q1: value IRF530 -> IRFZ44N
- R1: renamed from 100k1; value R -> 100k
Connections:
- net +12V: now also R2.1
- net GND: now also Q2.1 (E)
- new net: Q2.2 (B), R1.1, R3.2
- new net: A1.6 (D3), R3.1
- new net: Q1.1 (G), Q2.3 (C), R2.2
Other:
- moved on the sheet: J2, Q1, R1

Commit message: added 10uF at +5V output
Parts:
- added C1: 10uF, symbol Device:C_Polarized
Connections:
- net +5V: now also C1.1
- net GND: now also C1.2
Changed lines of the file:
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@@
 (kicad_sch (version 20230121) (generator eeschema)
   (paper "A4")
+  (junction (at 80.01 62.23) (diameter 0) (color 0 0 0 0)
+  )
   (junction (at 63.5 106.68) (diameter 0) (color 0 0 0 0)
   )
@@
     (stroke (width 0) (type default))
   )
+  (wire (pts (xy 80.01 62.23) (xy 81.28 62.23))
+    (stroke (width 0) (type default))
+  )
   (wire (pts (xy 116.84 116.84) (xy 127 116.84))
     (stroke (width 0) (type default))
   )
+  (wire (pts (xy 80.01 72.39) (xy 80.01 69.85))
+    (stroke (width 0) (type default))
+  )
   (wire (pts (xy 57.15 62.23) (xy 60.96 62.23))
     (stroke (width 0) (type default))
   )
-  (wire (pts (xy 76.2 62.23) (xy 81.28 62.23))
+  (wire (pts (xy 76.2 62.23) (xy 80.01 62.23))
     (stroke (width 0) (type default))
   )
@@
         (path "/df2671da-58c6-4dff-9178-ec59892716be"
           (reference "#PWR07") (unit 1)
+        )
+      )
+    )
+  )
+  (symbol (lib_id "power:GND") (at 80.01 72.39 0) (unit 1)
+    (in_bom yes) (on_board yes) (dnp no) (fields_autoplaced)
+    (property "Reference" "#PWR015" (at 80.01 78.74 0)
+      (effects (font (size 1.27 1.27)) hide)
+    )
+    (property "Value" "GND" (at 80.01 77.47 0)
+      (effects (font (size 1.27 1.27)))
+    )
+    (property "Footprint" "" (at 80.01 72.39 0)
+      (effects (font (size 1.27 1.27)) hide)
+    )
+    (property "Datasheet" "" (at 80.01 72.39 0)
+      (effects (font (size 1.27 1.27)) hide)
+    )
+    (pin "1")
+    (instances
+      (project "board"
+        (path "/df2671da-58c6-4dff-9178-ec59892716be"
+          (reference "#PWR015") (unit 1)
         )
       )
@@
         )
       )
+    )
+  )
+  (symbol (lib_id "Device:C_Polarized") (at 80.01 66.04 0) (unit 1)
+    (in_bom yes) (on_board yes) (dnp no) (fields_autoplaced)
+    (property "Reference" "C1" (at 83.82 63.881 0)
+      (effects (font (size 1.27 1.27)) (justify left))
+    )
+    (property "Value" "10uF" (at 83.82 66.421 0)
+      (effects (font (size 1.27 1.27)) (justify left))
+    )
+    (property "Footprint" "" (at 80.9752 69.85 0)
+      (effects (font (size 1.27 1.27)) hide)
+    )
+    (property "Datasheet" "~" (at 80.01 66.04 0)
+      (effects (font (size 1.27 1.27)) hide)
+    )
+    (pin "2")
+    (pin "1")
+    (instances
+      (project "board"
+        (path "/df2671da-58c6-4dff-9178-ec59892716be"
+          (reference "C1") (unit 1)
+        )
+      )
